Commit message: Update wheels.xacro

File: my_robot_urdf/urdf/wheels.xacro (robot description, xacro)
@@ -28,5 +28,5 @@
         <parent link="link_chassis"/>
         <axis rpy="0 0 0" xyz="0 1 0"/>
-        <limit effort="10000" velocity="1000"/>
+        <!--limit effort="10000" velocity="1000"/-->
         <joint_properties damping="1.0" friction="1.0"/>
       </joint>
@@ -37,3 +37,8 @@
                 izz="${mass*(r*r)/2}" />
     </xacro:macro>
+    <xacro:macro name="box_inertia" params="mass w h d">
+      <inertia  ixx="${mass*(h*h+d*d)/12}" ixy = "0" ixz = "0"
+                iyy="${mass*(w*w+d*d)/12}" iyz = "0"
+                izz="${mass*(w*w+h+h)/12}" />
+    </xacro:macro>
 </robot>
