Commit message: Update dd_urdf.xacro

File: my_robot_urdf/urdf/dd_urdf.xacro (robot description, xacro)
@@ -4,5 +4,6 @@
   <xacro:include filename="$(find my_robot_urdf)/urdf/dd_robot.gazebo" />
   <xacro:include filename="$(find my_robot_urdf)/urdf/wheels.xacro" />
-  <link name="link_chassis">
+  <static>false</static>
+<link name="link_chassis">
     <!-- pose and inertial -->
     <pose>0 0 0.1 0 0 0</pose>
@@ -15,5 +16,5 @@
     <collision name="collision_chassis">
       <geometry>
-        <cylinder radius="0.3" length="0.07"/>
+        <cylinder radius="0.3" length="0.05"/>
       </geometry>
     </collision>
@@ -21,13 +22,13 @@
       <origin rpy="0 0 0" xyz="0 0 0"/>
       <geometry>
-        <cylinder radius="0.3" length="0.07"/>
+        <cylinder radius="0.3" length="0.05"/>
       </geometry>
       <material name="blue"/>
     </visual>
-    <!-- caster front -->
+  <!-- caster front -->
     <collision name="caster_front_collision">
       <origin rpy=" 0 0 0" xyz="0.35 0 -0.05"/>
       <geometry>
-        <sphere radius="0.0325"/>
+        <sphere radius="0.05"/>
       </geometry>
       <surface>
@@ -42,31 +43,33 @@
       </surface>
     </collision>
-    <visual name="caster_front_visual">
-      <origin rpy=" 0 0 0" xyz="0.2 0 -0.0675"/>
+    <visual name="caster_front_wheel">
+      <origin rpy=" 0 0 0" xyz="0.2 0 -0.05"/>
       <geometry>
-        <sphere radius="0.0325"/>
+        <sphere radius="0.05"/>
       </geometry>
     </visual>
-  </link>
+    </link>
+  <!-- sensor_laser -->
   <link name="sensor_laser">
     <inertial>
       <origin xyz="0 0 0" rpy="0 0 0" />
       <mass value="1" />
-      <xacro:cylinder_inertia mass="1" r="0.05" l="0.1" />
+      <xacro:box_inertia mass="1" w="0.15" h="0.15" d="0.05" />
     </inertial>
     <visual>
       <origin xyz="0 0 0" rpy="0 0 0" />
       <geometry>
-        <box size="0.15 0.15 0.07"/>
+        <box size="0.15 0.15 0.05"/>
       </geometry>
       <material name="white" />
     </visual>
-    <collision>
+    <!--collision>
       <origin xyz="0 0 0" rpy="0 0 0"/>
       <geometry>
-        <box size="0.15 0.15 0.07"/>
+        <box size="0.15 0.15 0.05"/>
       </geometry>
-    </collision>
-  </link>
+    </collision -->
+    </link>
+   <!--  laser Joint -->
   <joint name="joint_sensor_laser" type="fixed">
     <origin xyz="0.15 0 0.05" rpy="0 0 0"/>
@@ -74,7 +77,9 @@
     <child link="sensor_laser"/>
   </joint>
+  <!-- right wheel and jt. -->
   <xacro:link_wheel name="link_right_wheel" />
   <xacro:joint_wheel name="joint_right_wheel" child="link_right_wheel" origin_xyz="0 -0.3 0" />
+  <!-- left wheel and jt. -->
   <xacro:link_wheel name="link_left_wheel" />
   <xacro:joint_wheel name="joint_left_wheel" child="link_left_wheel" origin_xyz="0 0.3 0" />
-</robot>
+    </robot>

Commit message: Update dd_urdf.xacro

File: my_robot_urdf/urdf/dd_urdf.xacro (robot description, xacro)
@@ -56,5 +56,5 @@
     <inertial>
       <origin xyz="0 0 0" rpy="0 0 0" />
-      <mass value="1" />
+      <mass value="3" />
       <xacro:box_inertia mass="1" w="0.15" h="0.15" d="0.05" />
     </inertial>
